File: Controller/V2/Controller.sch (KiCad schematic (older format))
At the start: 21 parts, among them J1 CONN_02X08, J10 CONN_01X02, J2 CONN_01X04, J3 CONN_01X02, J4 CONN_01X02, J5 CONN_01X02, J6 CONN_01X02, J7 CONN_01X02, J8 CONN_01X03, J9 CONN_01X02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

Commit message: Started to refactor code to use bettwe widget event handling Created UILib for use in future projects
Parts:
- removed J1: CONN_02X08, Connect:IDC_Header_Straight_16pins, symbol CONN_02X08
- added J1: CONN_02X05, Pin_Headers:Pin_Header_Straight_2x05_Pitch2.54mm, symbol CONN_02X05
- added J11, J12, J13: CONN_01X02, Pin_Headers:Pin_Header_Straight_1x02_Pitch2.54mm, symbol CONN_01X02
- added R2, R4: R, Resistors_ThroughHole:R_Axial_DIN0207_L6.3mm_D2.5mm_P7.62mm_Horizontal, symbol R
- added RV1: POT_TRIM, Potentiometers:Potentiometer_Trimmer_Bourns_3005, symbol POT_TRIM
- U1: symbol ARDUINO_NANO -> ARDUINO_NANO-RESCUE-Controller
Connections:
- net +5V: now also U5.9, J1.2 (P2), R2.2; no longer U5.2
- net AIN6: now also U1.21 (A2), J13.1 (P1); no longer U1.25 (A6)
- net GND: now also J8.3 (P3), J1.9 (P9), J11.2 (P2), J12.2 (P2), J13.2 (P2), R4.1; no longer J8.2 (P2)
- net IO2: now also J1.7 (P7)
- net IO3: now also J1.5 (P5)
- net IO4: now also J1.3 (P3)
- net IO5: now also J1.1 (P1)
- net IO6: now also J1.4 (P4)
- net IO7: now also J1.6 (P6)
- net IO8: now also J1.8 (P8)
- net IO9: now also J1.10 (P10)
- net RST_DDS: now also U1.20 (A1); no longer U1.19 (A0)
- net SEL_DAC_N: now also U1.25 (A6); no longer U1.13 (10)
- net VI_PEAK: now also U1.22 (A3); no longer U1.26 (A7)
- net VO_AMP: now also U3.8 (VOUTC), U5.1; no longer U3.6 (VOUTA), U5.10
- net VO_MOD_SEL: now also U1.26 (A7); no longer U1.21 (A2)
- net VO_RANGE: now also U1.13 (10/SS); no longer U1.22 (A3)
- net VO_REF0: now also J8.1 (P1), R4.2, RV1.3; no longer J8.3 (P3), U3.7 (VOUTB)
- net VO_REF1: now also J8.2 (P2), R2.1, RV1.1, RV1.2; no longer J8.1 (P1), U3.8 (VOUTC)
- net WR_DDS: now also U1.19 (A0); no longer U1.20 (A1)
- net at J7.1 (P1): now also U5.5; no longer U5.6
- net at J6.1 (P1): now also U5.10; no longer U5.1
- net at D1.2 (A), Q1.1 (D): now also U5.2; no longer U5.9
- new net VO_OFFSET: J11.1 (P1), U3.6 (VOUTA)
- new net VO_SWEEP: J12.1 (P1), U3.7 (VOUTB)
- no-connect marks 9 -> 10
Other:
- note added: "<- AIN"
- note added: "<- Modulation"
- note added: "<- Peak Detect"
- note added: "Modulation ->"
- note added: "Offset ->"
- note added: "Range Select ->"
- note added: "Ref ->"
- note added: "Sine ->"
- note added: "Square ->"
- note added: "Sweep ->"
- moved on the sheet: C3, J2, J5, J6, J8, U3
